Commit message: 1.1.1 Modify unit_factor2 value to 1e-6.

File: tm_description/cobot/tm5_700_description/xacro/macro.tm5-700-nominal.urdf.xacro (robot description, xacro)
@@ -64,5 +64,5 @@
     <xacro:property name="izz_5" value="${2643.21*unit_factor}" />
     <xacro:property name="izz_6" value="${1559.496*unit_factor}" />
-    <xacro:property name="unit_factor2" value="0.001"/>
+    <xacro:property name="unit_factor2" value="0.000001"/>
     <xacro:property name="cogx_1" value="${  0.0000000*unit_factor2}" />
     <xacro:property name="cogy_1" value="${  0.0000000*unit_factor2}" />

File: tm_description/cobot/tm5_700_description/xacro/macro.tm5x-700-nominal.urdf.xacro (robot description, xacro)
@@ -64,5 +64,5 @@
     <xacro:property name="izz_5" value="${2643.21*unit_factor}" />
     <xacro:property name="izz_6" value="${286.595*unit_factor}" />
-    <xacro:property name="unit_factor2" value="0.001"/>
+    <xacro:property name="unit_factor2" value="0.000001"/>
     <xacro:property name="cogx_1" value="${  0.0000000*unit_factor2}" />
     <xacro:property name="cogy_1" value="${  0.0000000*unit_factor2}" />

File: tm_description/cobot/tm5_900_description/xacro/macro.tm5x-900-nominal.urdf.xacro (robot description, xacro)
@@ -64,5 +64,5 @@
     <xacro:property name="izz_5" value="${2643.21*unit_factor}" />
     <xacro:property name="izz_6" value="${286.595*unit_factor}" />
-    <xacro:property name="unit_factor2" value="0.001"/>
+    <xacro:property name="unit_factor2" value="0.000001"/>
     <xacro:property name="cogx_1" value="${  0.0000000*unit_factor2}" />
     <xacro:property name="cogy_1" value="${  0.0000000*unit_factor2}" />

File: tm_description/cobot_s/tm12s_description/xacro/macro.tm12sft-nominal.urdf.xacro (robot description, xacro)
@@ -64,5 +64,5 @@
     <xacro:property name="izz_5" value="${3478.9518*unit_factor}" />
     <xacro:property name="izz_6" value="${3055.15940*unit_factor}" />
-    <xacro:property name="unit_factor2" value="0.001"/>
+    <xacro:property name="unit_factor2" value="0.000001"/>
     <xacro:property name="cogx_1" value="${ -1.0522458*unit_factor2}" />
     <xacro:property name="cogy_1" value="${ -5411.0119*unit_factor2}" />

File: tm_description/cobot_s/tm12s_description/xacro/macro.tm12sx-nominal.urdf.xacro (robot description, xacro)
@@ -64,5 +64,5 @@
     <xacro:property name="izz_5" value="${3478.9518*unit_factor}" />
     <xacro:property name="izz_6" value="${312.21304*unit_factor}" />
-    <xacro:property name="unit_factor2" value="0.001"/>
+    <xacro:property name="unit_factor2" value="0.000001"/>
     <xacro:property name="cogx_1" value="${ -1.0522458*unit_factor2}" />
     <xacro:property name="cogy_1" value="${ -5411.0119*unit_factor2}" />

File: tm_description/cobot_s/tm12s_description/xacro/macro.tm12sxft-nominal.urdf.xacro (robot description, xacro)
@@ -64,5 +64,5 @@
     <xacro:property name="izz_5" value="${3478.9518*unit_factor}" />
     <xacro:property name="izz_6" value="${1070.5771*unit_factor}" />
-    <xacro:property name="unit_factor2" value="0.001"/>
+    <xacro:property name="unit_factor2" value="0.000001"/>
     <xacro:property name="cogx_1" value="${ -1.0522458*unit_factor2}" />
     <xacro:property name="cogy_1" value="${ -5411.0119*unit_factor2}" />

File: tm_description/cobot_s/tm14s_description/xacro/macro.tm14s-nominal.urdf.xacro (robot description, xacro)
@@ -64,5 +64,5 @@
     <xacro:property name="izz_5" value="${3478.9518*unit_factor}" />
     <xacro:property name="izz_6" value="${1854.4783*unit_factor}" />
-    <xacro:property name="unit_factor2" value="0.001"/>
+    <xacro:property name="unit_factor2" value="0.000001"/>
     <xacro:property name="cogx_1" value="${ -1.0522458*unit_factor2}" />
     <xacro:property name="cogy_1" value="${ -5411.0119*unit_factor2}" />

File: tm_description/cobot_s/tm14s_description/xacro/macro.tm14sft-nominal.urdf.xacro (robot description, xacro)
@@ -64,5 +64,5 @@
     <xacro:property name="izz_5" value="${3478.9518*unit_factor}" />
     <xacro:property name="izz_6" value="${3055.15940*unit_factor}" />
-    <xacro:property name="unit_factor2" value="0.001"/>
+    <xacro:property name="unit_factor2" value="0.000001"/>
     <xacro:property name="cogx_1" value="${ -1.0522458*unit_factor2}" />
     <xacro:property name="cogy_1" value="${ -5411.0119*unit_factor2}" />

File: tm_description/cobot_s/tm14s_description/xacro/macro.tm14sx-nominal.urdf.xacro (robot description, xacro)
@@ -64,5 +64,5 @@
     <xacro:property name="izz_5" value="${3478.9518*unit_factor}" />
     <xacro:property name="izz_6" value="${312.21304*unit_factor}" />
-    <xacro:property name="unit_factor2" value="0.001"/>
+    <xacro:property name="unit_factor2" value="0.000001"/>
     <xacro:property name="cogx_1" value="${ -1.0522458*unit_factor2}" />
     <xacro:property name="cogy_1" value="${ -5411.0119*unit_factor2}" />

File: tm_description/cobot_s/tm14s_description/xacro/macro.tm14sxft-nominal.urdf.xacro (robot description, xacro)
@@ -64,5 +64,5 @@
     <xacro:property name="izz_5" value="${3478.9518*unit_factor}" />
     <xacro:property name="izz_6" value="${1070.5771*unit_factor}" />
-    <xacro:property name="unit_factor2" value="0.001"/>
+    <xacro:property name="unit_factor2" value="0.000001"/>
     <xacro:property name="cogx_1" value="${ -1.0522458*unit_factor2}" />
     <xacro:property name="cogy_1" value="${ -5411.0119*unit_factor2}" />

File: tm_description/cobot_s/tm20s_description/xacro/macro.tm20s-nominal.urdf.xacro (robot description, xacro)
@@ -64,5 +64,5 @@
     <xacro:property name="izz_5" value="${3478.9518*unit_factor}" />
     <xacro:property name="izz_6" value="${1854.4783*unit_factor}" />
-    <xacro:property name="unit_factor2" value="0.001"/>
+    <xacro:property name="unit_factor2" value="0.000001"/>
     <xacro:property name="cogx_1" value="${ -1.0522458*unit_factor2}" />
     <xacro:property name="cogy_1" value="${ -5411.0119*unit_factor2}" />

File: tm_description/cobot_s/tm20s_description/xacro/macro.tm20sft-nominal.urdf.xacro (robot description, xacro)
@@ -64,5 +64,5 @@
     <xacro:property name="izz_5" value="${3478.9518*unit_factor}" />
     <xacro:property name="izz_6" value="${3055.15940*unit_factor}" />
-    <xacro:property name="unit_factor2" value="0.001"/>
+    <xacro:property name="unit_factor2" value="0.000001"/>
     <xacro:property name="cogx_1" value="${ -1.0522458*unit_factor2}" />
     <xacro:property name="cogy_1" value="${ -5411.0119*unit_factor2}" />

File: tm_description/cobot_s/tm20s_description/xacro/macro.tm20sx-nominal.urdf.xacro (robot description, xacro)
@@ -64,5 +64,5 @@
     <xacro:property name="izz_5" value="${3478.9518*unit_factor}" />
     <xacro:property name="izz_6" value="${312.21304*unit_factor}" />
-    <xacro:property name="unit_factor2" value="0.001"/>
+    <xacro:property name="unit_factor2" value="0.000001"/>
     <xacro:property name="cogx_1" value="${ -1.0522458*unit_factor2}" />
     <xacro:property name="cogy_1" value="${ -5411.0119*unit_factor2}" />

File: tm_description/cobot_s/tm20s_description/xacro/macro.tm20sxft-nominal.urdf.xacro (robot description, xacro)
@@ -64,5 +64,5 @@
     <xacro:property name="izz_5" value="${3478.9518*unit_factor}" />
     <xacro:property name="izz_6" value="${1070.5771*unit_factor}" />
-    <xacro:property name="unit_factor2" value="0.001"/>
+    <xacro:property name="unit_factor2" value="0.000001"/>
     <xacro:property name="cogx_1" value="${ -1.0522458*unit_factor2}" />
     <xacro:property name="cogy_1" value="${ -5411.0119*unit_factor2}" />

File: tm_description/cobot_s/tm25s_description/xacro/macro.tm25sft-nominal.urdf.xacro (robot description, xacro)
@@ -64,5 +64,5 @@
     <xacro:property name="izz_5" value="${7195.1432*unit_factor}" />
     <xacro:property name="izz_6" value="${3055.1594*unit_factor}" />
-    <xacro:property name="unit_factor2" value="0.001"/>
+    <xacro:property name="unit_factor2" value="0.000001"/>
     <xacro:property name="cogx_1" value="${  0.0000000*unit_factor2}" />
     <xacro:property name="cogy_1" value="${ -7233.3847*unit_factor2}" />

File: tm_description/cobot_s/tm25s_description/xacro/macro.tm25sxft-nominal.urdf.xacro (robot description, xacro)
@@ -64,5 +64,5 @@
     <xacro:property name="izz_5" value="${7195.1432*unit_factor}" />
     <xacro:property name="izz_6" value="${1070.5771*unit_factor}" />
-    <xacro:property name="unit_factor2" value="0.001"/>
+    <xacro:property name="unit_factor2" value="0.000001"/>
     <xacro:property name="cogx_1" value="${  0.0000000*unit_factor2}" />
     <xacro:property name="cogy_1" value="${ -7233.3847*unit_factor2}" />

File: tm_description/cobot_s/tm30s_description/xacro/macro.tm30sft-nominal.urdf.xacro (robot description, xacro)
@@ -64,5 +64,5 @@
     <xacro:property name="izz_5" value="${7195.1432*unit_factor}" />
     <xacro:property name="izz_6" value="${3055.1594*unit_factor}" />
-    <xacro:property name="unit_factor2" value="0.001"/>
+    <xacro:property name="unit_factor2" value="0.000001"/>
     <xacro:property name="cogx_1" value="${  0.0000000*unit_factor2}" />
     <xacro:property name="cogy_1" value="${ -7233.3847*unit_factor2}" />

File: tm_description/cobot_s/tm30s_description/xacro/macro.tm30sxft-nominal.urdf.xacro (robot description, xacro)
@@ -64,5 +64,5 @@
     <xacro:property name="izz_5" value="${7195.1432*unit_factor}" />
     <xacro:property name="izz_6" value="${1070.5771*unit_factor}" />
-    <xacro:property name="unit_factor2" value="0.001"/>
+    <xacro:property name="unit_factor2" value="0.000001"/>
     <xacro:property name="cogx_1" value="${  0.0000000*unit_factor2}" />
     <xacro:property name="cogy_1" value="${ -7233.3847*unit_factor2}" />

File: tm_description/cobot_s/tm5s_description/xacro/macro.tm5s-nominal.urdf.xacro (robot description, xacro)
@@ -64,5 +64,5 @@
     <xacro:property name="izz_5" value="${3478.9518*unit_factor}" />
     <xacro:property name="izz_6" value="${1854.4783*unit_factor}" />
-    <xacro:property name="unit_factor2" value="0.001"/>
+    <xacro:property name="unit_factor2" value="0.000001"/>
     <xacro:property name="cogx_1" value="${-0.95125746*unit_factor2}" />
     <xacro:property name="cogy_1" value="${ -4841.5002*unit_factor2}" />

File: tm_description/cobot_s/tm5s_description/xacro/macro.tm5sft-nominal.urdf.xacro (robot description, xacro)
@@ -64,5 +64,5 @@
     <xacro:property name="izz_5" value="${3478.9518*unit_factor}" />
     <xacro:property name="izz_6" value="${3055.15940*unit_factor}" />
-    <xacro:property name="unit_factor2" value="0.001"/>
+    <xacro:property name="unit_factor2" value="0.000001"/>
     <xacro:property name="cogx_1" value="${-0.95125746*unit_factor2}" />
     <xacro:property name="cogy_1" value="${ -4841.5002*unit_factor2}" />
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