Commit message: 1.3.0 fix: correct `cogx_3` parameter value for TM7S series LINK3.

File: tm_description/cobot_s/tm7s_description/xacro/macro.tm7s-nominal.urdf.xacro (robot description, xacro)
@@ -71,5 +71,5 @@
     <xacro:property name="cogy_2" value="${  0.0000000*unit_factor2}" />
     <xacro:property name="cogz_2" value="${ -150758.58*unit_factor2}" />
-    <xacro:property name="cogx_3" value="${ 2203387.78*unit_factor2}" />
+    <xacro:property name="cogx_3" value="${  220338.78*unit_factor2}" /> <!-- MC-002: modify  -->
     <xacro:property name="cogy_3" value="${  2.4404199*unit_factor2}" />
     <xacro:property name="cogz_3" value="${  22677.955*unit_factor2}" />

File: tm_description/cobot_s/tm7s_description/xacro/macro.tm7sft-nominal.urdf.xacro (robot description, xacro)
@@ -71,5 +71,5 @@
     <xacro:property name="cogy_2" value="${  0.0000000*unit_factor2}" />
     <xacro:property name="cogz_2" value="${ -150758.58*unit_factor2}" />
-    <xacro:property name="cogx_3" value="${ 2203387.78*unit_factor2}" />
+    <xacro:property name="cogx_3" value="${  220338.78*unit_factor2}" /> <!-- MC-002: modify  -->
     <xacro:property name="cogy_3" value="${  2.4404199*unit_factor2}" />
     <xacro:property name="cogz_3" value="${  22677.955*unit_factor2}" />

File: tm_description/cobot_s/tm7s_description/xacro/macro.tm7sx-nominal.urdf.xacro (robot description, xacro)
@@ -71,5 +71,5 @@
     <xacro:property name="cogy_2" value="${  0.0000000*unit_factor2}" />
     <xacro:property name="cogz_2" value="${ -150758.58*unit_factor2}" />
-    <xacro:property name="cogx_3" value="${ 2203387.78*unit_factor2}" />
+    <xacro:property name="cogx_3" value="${  220338.78*unit_factor2}" /> <!-- MC-002: modify  -->
     <xacro:property name="cogy_3" value="${  2.4404199*unit_factor2}" />
     <xacro:property name="cogz_3" value="${  22677.955*unit_factor2}" />

File: tm_description/cobot_s/tm7s_description/xacro/macro.tm7sxft-nominal.urdf.xacro (robot description, xacro)
@@ -71,5 +71,5 @@
     <xacro:property name="cogy_2" value="${  0.0000000*unit_factor2}" />
     <xacro:property name="cogz_2" value="${ -150758.58*unit_factor2}" />
-    <xacro:property name="cogx_3" value="${ 2203387.78*unit_factor2}" />
+    <xacro:property name="cogx_3" value="${  220338.78*unit_factor2}" /> <!-- MC-002: modify  -->
     <xacro:property name="cogy_3" value="${  2.4404199*unit_factor2}" />
     <xacro:property name="cogz_3" value="${  22677.955*unit_factor2}" />
