Commit message: 1.4.0 fix: correct the parameter values ​​`cogx_3,cogy_3,cogz_3` for TM6S series LINK3.

File: tm_description/cobot_s/tm6s_description/xacro/macro.tm6s-nominal.urdf.xacro (robot description, xacro)
@@ -71,7 +71,7 @@
     <xacro:property name="cogy_2" value="${  0.0000000*unit_factor2}" />
     <xacro:property name="cogz_2" value="${ -182283.92*unit_factor2}" />
-    <xacro:property name="cogx_3" value="${  1.6047637*unit_factor2}" />
-    <xacro:property name="cogy_3" value="${ -544.92737*unit_factor2}" />
-    <xacro:property name="cogz_3" value="${ -55316.774*unit_factor2}" />
+    <xacro:property name="cogx_3" value="${  518282.63*unit_factor2}" />
+    <xacro:property name="cogy_3" value="${  1.6047637*unit_factor2}" />
+    <xacro:property name="cogz_3" value="${ -54492.737*unit_factor2}" />
     <xacro:property name="cogx_4" value="${ -3.6473102*unit_factor2}" />
     <xacro:property name="cogy_4" value="${ -6381.2605*unit_factor2}" />

File: tm_description/cobot_s/tm6s_description/xacro/macro.tm6sft-nominal.urdf.xacro (robot description, xacro)
@@ -71,7 +71,7 @@
     <xacro:property name="cogy_2" value="${  0.0000000*unit_factor2}" />
     <xacro:property name="cogz_2" value="${ -182283.92*unit_factor2}" />
-    <xacro:property name="cogx_3" value="${  1.6047637*unit_factor2}" />
-    <xacro:property name="cogy_3" value="${ -544.92737*unit_factor2}" />
-    <xacro:property name="cogz_3" value="${ -55316.774*unit_factor2}" />
+    <xacro:property name="cogx_3" value="${  518282.63*unit_factor2}" />
+    <xacro:property name="cogy_3" value="${  1.6047637*unit_factor2}" />
+    <xacro:property name="cogz_3" value="${ -54492.737*unit_factor2}" />
     <xacro:property name="cogx_4" value="${ -3.6473102*unit_factor2}" />
     <xacro:property name="cogy_4" value="${ -6381.2605*unit_factor2}" />

File: tm_description/cobot_s/tm6s_description/xacro/macro.tm6sx-nominal.urdf.xacro (robot description, xacro)
@@ -71,7 +71,7 @@
     <xacro:property name="cogy_2" value="${  0.0000000*unit_factor2}" />
     <xacro:property name="cogz_2" value="${ -182283.92*unit_factor2}" />
-    <xacro:property name="cogx_3" value="${  1.6047637*unit_factor2}" />
-    <xacro:property name="cogy_3" value="${ -544.92737*unit_factor2}" />
-    <xacro:property name="cogz_3" value="${ -55316.774*unit_factor2}" />
+    <xacro:property name="cogx_3" value="${  518282.63*unit_factor2}" />
+    <xacro:property name="cogy_3" value="${  1.6047637*unit_factor2}" />
+    <xacro:property name="cogz_3" value="${ -54492.737*unit_factor2}" />
     <xacro:property name="cogx_4" value="${ -3.6473102*unit_factor2}" />
     <xacro:property name="cogy_4" value="${ -6381.2605*unit_factor2}" />

File: tm_description/cobot_s/tm6s_description/xacro/macro.tm6sxft-nominal.urdf.xacro (robot description, xacro)
@@ -71,7 +71,7 @@
     <xacro:property name="cogy_2" value="${  0.0000000*unit_factor2}" />
     <xacro:property name="cogz_2" value="${ -182283.92*unit_factor2}" />
-    <xacro:property name="cogx_3" value="${  1.6047637*unit_factor2}" />
-    <xacro:property name="cogy_3" value="${ -544.92737*unit_factor2}" />
-    <xacro:property name="cogz_3" value="${ -55316.774*unit_factor2}" />
+    <xacro:property name="cogx_3" value="${  518282.63*unit_factor2}" />
+    <xacro:property name="cogy_3" value="${  1.6047637*unit_factor2}" />
+    <xacro:property name="cogz_3" value="${ -54492.737*unit_factor2}" />
     <xacro:property name="cogx_4" value="${ -3.6473102*unit_factor2}" />
     <xacro:property name="cogy_4" value="${ -6381.2605*unit_factor2}" />
